Commit message: lws updated urdf and keyboard control added

File: ros2_ws/src/lws_description/urdf/common_properties.xacro (robot description, xacro)
@@ -1,9 +1,18 @@
 <?xml version="1.0"?>
 <robot xmlns:xacro="http://www.ros.org/wiki/xacro">
-    <material name="green">
-        <color rgba="0 0.6 0 1" />
+    <material name="steel_gray">
+        <color rgba="0.7 0.7 0.7 1.0"/>
     </material>
-    <material name="gray">
-        <color rgba="0.7 0.7 0.7 1" />
+    <material name="dark_gray">
+      <color rgba="0.3 0.3 0.3 1.0"/>
+    </material>
+    <material name="black">
+      <color rgba="0.1 0.1 0.1 1.0"/>
+    </material>
+    <material name="red">
+      <color rgba="0.8 0.1 0.1 1.0"/>
+    </material>
+    <material name="blue">
+      <color rgba="0.1 0.1 0.8 1.0"/>
     </material>
     <xacro:macro name="box_inertia" params="m x y z o_xyz o_rpy">

File: ros2_ws/src/lws_description/urdf/lws.urdf.xacro (robot description, xacro)
@@ -5,3 +5,4 @@
     <xacro:include filename="$(find lws_description)/urdf/lws_base.xacro" />
     <xacro:include filename="$(find lws_description)/urdf/lws_base_gz.xacro" />
+    <xacro:include filename="$(find lws_description)/urdf/camera.xacro" />
 </robot>

File: ros2_ws/src/lws_description/urdf/lws_base.xacro (robot description, xacro)
@@ -2,48 +2,104 @@
 <robot name="lws"
     xmlns:xacro="http://www.ros.org/wiki/xacro">
-    <!-- Основна база -->
+    <xacro:property name="base_length" value="2" />
+    <xacro:property name="base_width" value="2" />
+    <xacro:property name="base_height" value="0.5" />
+    <xacro:property name="turret_base_radius" value="${base_width / 4}" />
+    <xacro:property name="turret_base_length" value="${base_height / 1.75}" />
+    <xacro:property name="turret_head_radius" value="${turret_base_radius / 8}" />
+    <xacro:property name="turret_head_length" value="${1.5 * turret_base_radius}" />
     <link name="base_link">
         <visual>
             <geometry>
-                <box size="0.1 0.1 0.05"/>
+                <box size="${base_length} ${base_width} ${base_height}"/>
+            </geometry>
+            <origin xyz="0 0 ${base_height / 2.0}" rpy="0 0 0" />
+            <material name="red" />
+        </visual>
+        <collision>
+            <geometry>
+                <box size="${base_length} ${base_width} ${base_height}"/>
+            </geometry>
+            <origin xyz="0 0 ${base_height / 2.0}" rpy="0 0 0" />
+        </collision>
+        <xacro:box_inertia m="50.0" x="${base_length}" y="${base_width}" z="${base_height}"
+                           o_xyz="0 0 0" o_rpy="0 0 0" />
+    </link>
+    <link name="turret_base_link">
+        <visual>
+            <geometry>
+                <cylinder radius="${turret_base_radius}" length="${turret_base_length}"/>
             </geometry>
             <origin xyz="0 0 0" rpy="0 0 0" />
-            <material name="grey">
-                <color rgba="0.5 0.5 0.5 1.0"/>
-            </material>
+            <material name="dark_gray" />
         </visual>
+        <!-- <collision>
+            <geometry>
+                <cylinder radius="${turret_base_radius}" length="${turret_base_length}"/>
+            </geometry>
+            <origin xyz="0 0 0" rpy="0 0 0" />
+        </collision> -->
+        <xacro:cylinder_inertia m="12.5" r="${turret_base_radius}" l="${turret_base_length}"
+                                    o_xyz="0 0 0" o_rpy="0 0 0" />
     </link>
-    <link name="platform">
+    <joint name="base_turret_base_joint" type="revolute">
+        <parent link="base_link"/>
+        <child link="turret_base_link"/>
+        <origin xyz="0 0 ${base_height + turret_base_length / 2.0}" rpy="0 0 ${- pi / 4.0}"/>
+        <axis xyz="0 0 1"/>
+        <limit
+            lower="${-40 * pi / 180.0}"
+            upper="${40 * pi / 180.0}"
+            effort="10.0"
+            velocity="1.0"/>
+        <dynamics damping="0.7" friction="0.0"/>
+    </joint>
+<!--
+    <transmission name="base_turret_base_trans">
+        <type>transmission_interface/SimpleTransmission</type>
+        <joint name="base_turret_base_joint">
+            <hardwareInterface>hardware_interface/PositionJointInterface</hardwareInterface>
+        </joint>
+        <actuator name="base_turret_base_motor">
+            <mechanicalReduction>1</mechanicalReduction>
+        </actuator>
+    </transmission> -->
+    <link name="turret_head_link">
         <visual>
             <geometry>
-                <cylinder radius="0.05" length="0.02"/>
+                <cylinder radius="${turret_head_radius}" length="${turret_head_length}"/>
             </geometry>
-            <material name="dark_grey">
-                <color rgba="0.3 0.3 0.3 1.0"/>
-            </material>
+            <origin xyz="0 0 ${turret_head_length / 2.0}" rpy="0 0 0" />
+            <material name="dark_gray" />
         </visual>
+        <!-- <collision>
+            <geometry>
+                <cylinder radius="${turret_head_radius}" length="${turret_head_length}"/>
+            </geometry>
+            <origin xyz="0 0 ${turret_base_radius}" rpy="0 0 0" />
+        </collision> -->
+        <xacro:cylinder_inertia m="6.25" r="${turret_head_radius}" l="${turret_head_radius}"
+                                    o_xyz="0 0 0" o_rpy="0 0 0" />
     </link>
-    <joint name="base_to_platform" type="continuous">
-        <parent link="base_link"/>
-        <child link="platform"/>
-        <origin xyz="0 0 0.05" rpy="0 0 0"/>
-        <axis xyz="0 0 1"/>
+    <joint name="base_turret_head_joint" type="revolute">
+        <parent link="turret_base_link"/>
+        <child link="turret_head_link"/>
+        <origin xyz="0 0 0" rpy="0 ${pi / 2.0} ${pi / 4.0}"/>
+        <axis xyz="0 1 0"/>
+        <limit
+            lower="${-45 * pi / 180.0}"
+            upper="0"
+            effort="10.0"
+            velocity="1.0"/>
+        <dynamics damping="0.7" friction="0.0"/>
     </joint>
-    <link name="laser">
-        <visual>
-            <geometry>
-                <cylinder radius="0.02" length="0.1"/>
-            </geometry>
-            <material name="red">
-                <color rgba="1.0 0.0 0.0 1.0"/>
-            </material>
-        </visual>
-    </link>
-    <joint name="platform_to_laser" type="revolute">
-        <parent link="platform"/>
-        <child link="laser"/>
-        <origin xyz="0 0 0.02" rpy="0 0 0"/>
-        <axis xyz="1 0 0"/>
-        <limit lower="-0.5" upper="0.5" effort="1.0" velocity="0.5"/>
-    </joint>
+    <!-- <transmission name="base_turret_head_trans">
+        <type>transmission_interface/SimpleTransmission</type>
+        <joint name="base_turret_head_joint">
+            <hardwareInterface>hardware_interface/PositionJointInterface</hardwareInterface>
+        </joint>
+        <actuator name="base_turret_head_motor">
+            <mechanicalReduction>1</mechanicalReduction>
+        </actuator>
+    </transmission> -->
 </robot>

File: ros2_ws/src/lws_description/urdf/lws_base_gz.xacro (robot description, xacro)
@@ -7,3 +7,29 @@
         </plugin>
     </gazebo>
+    <gazebo>
+        <plugin filename="gz-sim-joint-position-controller-system" name="gz::sim::systems::JointPositionController">
+            <joint_name>base_turret_base_joint</joint_name>
+            <topic>turret_base_position_cmd</topic>
+            <p_gain>10.0</p_gain>
+            <i_gain>0.1</i_gain>
+            <d_gain>1.0</d_gain>
+            <i_max>1.0</i_max>
+            <i_min>-1.0</i_min>
+            <cmd_max>10.0</cmd_max>
+            <cmd_min>-10.0</cmd_min>
+        </plugin>
+    </gazebo>
+    <gazebo>
+        <plugin filename="gz-sim-joint-position-controller-system" name="gz::sim::systems::JointPositionController">
+            <joint_name>base_turret_head_joint</joint_name>
+            <topic>turret_head_position_cmd</topic>
+            <p_gain>10.0</p_gain>
+            <i_gain>0.1</i_gain>
+            <d_gain>1.0</d_gain>
+            <i_max>1.0</i_max>
+            <i_min>-1.0</i_min>
+            <cmd_max>10.0</cmd_max>
+            <cmd_min>-10.0</cmd_min>
+        </plugin>
+    </gazebo>
 </robot>
